Commit message: fix(comments): Remove unnecessary comments

File: assignments_personal_ws/src/vw-assign1-2025-parol6-mesh-pkg/urdf/PAROL6.urdf.xacro (robot description, xacro)
@@ -26,5 +26,4 @@
       <geometry>
         <box size="0.23 0.12 0.06" />
-        <!-- <mesh filename="package://vw-assign1-2025-parol6-fixed-pkg/meshes/base_link.STL" /> -->
       </geometry>
     </collision>
@@ -49,6 +48,4 @@
       <geometry>
         <cylinder radius="0.05" length="0.05" />
-        <!-- <box size="0.1 0.22 0.075" /> -->
-        <!-- <mesh filename="package://vw-assign1-2025-parol6-fixed-pkg/meshes/L1.STL" /> -->
       </geometry>
     </collision>
@@ -80,5 +77,4 @@
       <geometry>
         <cylinder radius="0.03" length="0.2" />
-        <!-- <mesh filename="package://vw-assign1-2025-parol6-fixed-pkg/meshes/L2.STL" /> -->
       </geometry>
     </collision>
@@ -110,5 +106,4 @@
       <geometry>
         <box size="0.1 0.11 0.07" />
-        <!-- <mesh filename="package://vw-assign1-2025-parol6-fixed-pkg/meshes/L3.STL" /> -->
       </geometry>
     </collision>
@@ -140,5 +135,4 @@
       <geometry>
         <box size="0.07 0.06 0.050" />
-        <!-- <mesh filename="package://vw-assign1-2025-parol6-fixed-pkg/meshes/L4.STL" /> -->
       </geometry>
     </collision>
@@ -170,5 +164,4 @@
       <geometry>
         <cylinder radius="0.03" length="0.08" />
-        <!-- <mesh filename="package://vw-assign1-2025-parol6-fixed-pkg/meshes/L5.STL" /> -->
       </geometry>
     </collision>
@@ -200,5 +193,4 @@
       <geometry>
         <box size="0.08 0.05 0.04" />
-        <!-- <mesh filename="package://vw-assign1-2025-parol6-fixed-pkg/meshes/L6.STL" /> -->
       </geometry>
     </collision>
