Commit message: feat(assign1): Finis Part 2a

File: assignments_personal_ws/src/vw-assign1-2025-parol6-fixed-pkg/urdf/PAROL6.urdf.xacro (robot description, xacro)
@@ -5,6 +5,10 @@
     <parent link="world"/>
     <child link="base_link"/>
+    <!-- <child link="base_conn_4"/> -->
     <origin rpy="0 0 0" xyz="0.0 0.0 0.00"/>
   </joint>
+<!-- ================================ -->
+<!--             ROBOT                -->
+<!-- ================================ -->
   <link name="base_link">
     <inertial>
@@ -294,3 +298,114 @@
     <selfCollide>true</selfCollide>
   </gazebo>
+  <!-- ================================ -->
+  <!--            CONNECT 4             -->
+  <!-- ================================ -->
+  <link name="base_conn_4">
+    <visual>
+      <origin xyz="0 0 0" rpy="0 0 0" />
+      <geometry>
+        <mesh filename="package://vw-assign1-2025-parol6-fixed-pkg/meshes/base_conn_4.STL" scale="0.001 0.001 0.001"/>
+      </geometry>
+      <material name="">
+        <color rgba="0 1 0 1" />
+      </material>
+    </visual>
+    <collision>
+      <origin xyz="0 0 0" rpy="0 0 0" />
+      <geometry>
+        <mesh filename="package://vw-assign1-2025-parol6-fixed-pkg/meshes/base_conn_4.STL" scale="0.001 0.001 0.001"/>
+      </geometry>
+    </collision>
+    <inertial>
+      <mass value="1.0" />
+      <origin xyz="0 0 0" />
+      <inertia ixx="1.0" ixy="0.0" ixz="0.0" iyy="1.0" iyz="0.0" izz="1.0" />
+    </inertial>
+  </link>
+  <link name="board_conn_4">
+    <visual>
+      <origin xyz="0 0 0" rpy="0 0 0" />
+      <geometry>
+        <mesh filename="package://vw-assign1-2025-parol6-fixed-pkg/meshes/board_conn_4.STL" scale="0.001 0.001 0.001"/>
+      </geometry>
+      <material name="">
+        <color rgba="0 0 1 1" />
+      </material>
+    </visual>
+    <collision>
+      <origin xyz="0 0 0" rpy="0 0 0" />
+      <geometry>
+        <mesh filename="package://vw-assign1-2025-parol6-fixed-pkg/meshes/board_conn_4.STL" scale="0.001 0.001 0.001"/>
+      </geometry>
+    </collision>
+    <inertial>
+      <mass value="1.0" />
+      <origin xyz="0 0 0" />
+      <inertia ixx="1.0" ixy="0.0" ixz="0.0" iyy="1.0" iyz="0.0" izz="1.0" />
+    </inertial>
+  </link>
+  <link name="coin_holder">
+    <visual>
+      <origin xyz="0 0 0" rpy="0 0 0" />
+      <geometry>
+        <mesh filename="package://vw-assign1-2025-parol6-fixed-pkg/meshes/muntjes_houder.STL" scale="0.001 0.001 0.001"/>
+      </geometry>
+      <material name="">
+        <color rgba="1.0 1.0 0.0 1" />
+      </material>
+    </visual>
+    <collision>
+      <origin xyz="0 0 0" rpy="0 0 0" />
+      <geometry>
+        <mesh filename="package://vw-assign1-2025-parol6-fixed-pkg/meshes/muntjes_houder.STL" scale="0.001 0.001 0.001"/>
+      </geometry>
+    </collision>
+    <inertial>
+      <mass value="1.0" />
+      <origin xyz="0 0 0" />
+      <inertia ixx="1.0" ixy="0.0" ixz="0.0" iyy="1.0" iyz="0.0" izz="1.0" />
+    </inertial>
+  </link>
+  <link name="coin">
+    <visual>
+      <origin xyz="0 0 0" rpy="0 0 0" />
+      <geometry>
+        <mesh filename="package://vw-assign1-2025-parol6-fixed-pkg/meshes/muntje.STL" scale="0.001 0.001 0.001"/>
+      </geometry>
+      <material name="">
+        <color rgba="1 1 1 1" />
+      </material>
+    </visual>
+    <collision>
+      <origin xyz="0 0 0" rpy="0 0 0" />
+      <geometry>
+        <mesh filename="package://vw-assign1-2025-parol6-fixed-pkg/meshes/muntje.STL" scale="0.001 0.001 0.001"/>
+      </geometry>
+    </collision>
+    <inertial>
+      <mass value="1.0" />
+      <origin xyz="0 0 0" />
+      <inertia ixx="1.0" ixy="0.0" ixz="0.0" iyy="1.0" iyz="0.0" izz="1.0" />
+    </inertial>
+  </link>
+  <joint name="joint_base_conn_4_world" type="fixed">
+    <parent link="world"/>
+    <child link="base_conn_4"/>
+    <origin xyz="0.30 0 0.00" rpy="0 0 0"/>
+  </joint>
+  <joint name="joint_board_conn_4_world" type="fixed">
+    <parent link="world"/>
+    <child link="board_conn_4"/>
+    <origin xyz="0.581 0.031 0.006" rpy="0 0 -0.226"/>
+  </joint>
+  <joint name="joint_coin_holder_world" type="fixed">
+    <parent link="world"/>
+    <child link="coin_holder"/>
+    <origin xyz="0.30 0.08 0.00" rpy="1.574 0 0"/>
+  </joint>
+  <joint name="joint_coin_world" type="fixed">
+    <parent link="world"/>
+    <child link="coin"/>
+    <origin xyz="0.34 0.08 0.00" rpy="0 0 0"/>
+  </joint>
 </robot>

Commit message: fix(collision): Remove comments and add simple collision to the coin

File: assignments_personal_ws/src/vw-assign1-2025-parol6-fixed-pkg/urdf/PAROL6.urdf.xacro (robot description, xacro)
@@ -5,5 +5,4 @@
     <parent link="world"/>
     <child link="base_link"/>
-    <!-- <child link="base_conn_4"/> -->
     <origin rpy="0 0 0" xyz="0.0 0.0 0.00"/>
   </joint>
@@ -30,5 +29,4 @@
       <geometry>
         <box size="0.23 0.12 0.06" />
-        <!-- <mesh filename="package://vw-assign1-2025-parol6-fixed-pkg/meshes/base_link.STL" /> -->
       </geometry>
     </collision>
@@ -53,6 +51,4 @@
       <geometry>
         <cylinder radius="0.05" length="0.05" />
-        <!-- <box size="0.1 0.22 0.075" /> -->
-        <!-- <mesh filename="package://vw-assign1-2025-parol6-fixed-pkg/meshes/L1.STL" /> -->
       </geometry>
     </collision>
@@ -84,5 +80,4 @@
       <geometry>
         <cylinder radius="0.03" length="0.2" />
-        <!-- <mesh filename="package://vw-assign1-2025-parol6-fixed-pkg/meshes/L2.STL" /> -->
       </geometry>
     </collision>
@@ -114,5 +109,4 @@
       <geometry>
         <box size="0.1 0.11 0.07" />
-        <!-- <mesh filename="package://vw-assign1-2025-parol6-fixed-pkg/meshes/L3.STL" /> -->
       </geometry>
     </collision>
@@ -144,5 +138,4 @@
       <geometry>
         <box size="0.07 0.06 0.050" />
-        <!-- <mesh filename="package://vw-assign1-2025-parol6-fixed-pkg/meshes/L4.STL" /> -->
       </geometry>
     </collision>
@@ -174,5 +167,4 @@
       <geometry>
         <cylinder radius="0.03" length="0.08" />
-        <!-- <mesh filename="package://vw-assign1-2025-parol6-fixed-pkg/meshes/L5.STL" /> -->
       </geometry>
     </collision>
@@ -204,5 +196,4 @@
       <geometry>
         <box size="0.08 0.05 0.04" />
-        <!-- <mesh filename="package://vw-assign1-2025-parol6-fixed-pkg/meshes/L6.STL" /> -->
       </geometry>
     </collision>
@@ -378,7 +369,7 @@
     </visual>
     <collision>
-      <origin xyz="0 0 0" rpy="0 0 0" />
-      <geometry>
-        <mesh filename="package://vw-assign1-2025-parol6-fixed-pkg/meshes/muntje.STL" scale="0.001 0.001 0.001"/>
+      <origin xyz="0.0170 0.0170 0.006" rpy="0 0 0" />
+      <geometry>
+        <cylinder radius="0.0165" length="0.010" />
       </geometry>
     </collision>

File: assignments_personal_ws/src/vw-assign1-2025-parol6-static-pkg/urdf/connect4.urdf.xacro (robot description, xacro)
@@ -15,5 +15,4 @@
       </geometry>
     </collision>
-    <!-- <inertial><mass value="1"/><origin xyz="0 0 0"/><inertia ixx="1" iyy="1" izz="1" ixy="0" ixz="0" iyz="0"/></inertial> -->
   </link>
   <link name="board_conn_4">
@@ -31,5 +30,4 @@
       </geometry>
     </collision>
-    <!-- <inertial><mass value="1"/><origin xyz="0 0 0"/><inertia ixx="1" iyy="1" izz="1" ixy="0" ixz="0" iyz="0"/></inertial> -->
   </link>
   <link name="coin_holder">
@@ -47,5 +45,4 @@
       </geometry>
     </collision>
-    <!-- <inertial><mass value="0.5"/><origin xyz="0 0 0"/><inertia ixx="1" iyy="1" izz="1" ixy="0" ixz="0" iyz="0"/></inertial> -->
   </link>
   <link name="coin">
@@ -59,11 +56,11 @@
     </visual>
     <collision>
+      <origin xyz="0.0170 0.0170 0.006" rpy="0 0 0" />
       <geometry>
-        <mesh filename="package://vw-assign1-2025-parol6-fixed-pkg/meshes/muntje.STL" scale="0.001 0.001 0.001"/>
+        <cylinder radius="0.0165" length="0.010" />
       </geometry>
     </collision>
-    <!-- <inertial><mass value="0.1"/><origin xyz="0 0 0"/><inertia ixx="0.01" iyy="0.01" izz="0.01" ixy="0" ixz="0" iyz="0"/></inertial> -->
   </link>
-  Fix all parts to base_conn_4; adjust relative poses
+  <!-- Fix all parts to base_conn_4; adjust relative poses -->
   <joint name="board_to_base" type="fixed">
     <parent link="base_conn_4"/>
